File: c5_adapter/kicad/c5_adapter.kicad_sch (KiCad schematic)
At the start: 7 parts, among them J1 Conn_01x10, J2 Conn_01x10, SW1 SW_DPDT_x2, SW2 SW_DPDT_x2, U1 ESP32-C5-DevKitC-1

Commit message: Code refactoring
Parts:
- added IC1: TLV6700DDCR, TLV6700DDCR:SOT95P280X110-6N, symbol TLV6700DDCR:TLV6700DDCR
Connections:
- net RST: now reaches U1.2 (EN/RESET)
- no-connect marks 3 -> 2
Changed lines of the file:
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@@
 	(paper "A4")
 	(no_connect
-		(at 137.16 55.88)
-	)
-	(no_connect
 		(at 69.85 36.83)
 	)
@@
 		(pts
 			(xy 133.35 86.36) (xy 137.16 86.36)
+		)
+		(stroke
+			(width 0)
+			(type default)
+		)
+	)
+	(wire
+		(pts
+			(xy 133.35 55.88) (xy 137.16 55.88)
 		)
 		(stroke
@@
 				)
 				(justify left)
+				(hide yes)
+			)
+		)
+	)
+	(global_label "RST"
+		(shape input)
+		(at 133.35 55.88 180)
+		(fields_autoplaced yes)
+		(effects
+			(font
+				(size 1.27 1.27)
+			)
+			(justify right)
+		)
+		(property "Intersheetrefs" "${INTERSHEET_REFS}"
+			(at 126.9177 55.88 0)
+			(effects
+				(font
+					(size 1.27 1.27)
+				)
+				(justify right)
 				(hide yes)
 			)
@@
 					(unit 1)
 				)
+			)
+		)
+	)
+	(symbol
+		(lib_id "TLV6700DDCR:TLV6700DDCR")
+		(at 81.28 49.53 0)
+		(unit 1)
+		(exclude_from_sim no)
+		(in_bom yes)
+		(on_board yes)
+		(dnp no)
+		(fields_autoplaced yes)
+		(property "Reference" "IC1"
+			(at 95.25 41.91 0)
+			(effects
+				(font
+					(size 1.27 1.27)
+				)
+			)
+		)
+		(property "Value" "TLV6700DDCR"
+			(at 95.25 44.45 0)
+			(effects
+				(font
+					(size 1.27 1.27)
+				)
+			)
+		)
+		(property "Footprint" "TLV6700DDCR:SOT95P280X110-6N"
+			(at 105.41 144.45 0)
+			(effects
+				(font
+					(size 1.27 1.27)
+				)
+				(justify left top)
+				(hide yes)
+			)
+		)
+		(property "Datasheet" "http://www.ti.com/lit/gpn/tlv6700"
+			(at 105.41 244.45 0)
+			(effects
+				(font
+					(size 1.27 1.27)
+				)
+				(justify left top)
+				(hide yes)
+			)
+		)
+		(property "Description" "TLV6700 Micropower, 18V Window Comparator with 400mV Reference"
+			(at 81.28 49.53 0)
+			(effects
+				(font
+					(size 1.27 1.27)
+				)
+				(hide yes)
+			)
+		)
+		(property "Height" "1.1"
+			(at 105.41 444.45 0)
+			(effects
+				(font
+					(size 1.27 1.27)
+				)
+				(justify left top)
+				(hide yes)
+			)
+		)
+		(property "Mouser Part Number" "595-TLV6700DDCR"
+			(at 105.41 544.45 0)
+			(effects
+				(font
+					(size 1.27 1.27)
+				)
+				(justify left top)
+				(hide yes)
+			)
+		)
+		(property "Mouser Price/Stock" "https://www.mouser.co.uk/ProductDetail/Texas-Instruments/TLV6700DDCR?qs=r5DSvlrkXmIgfUTYRQlC3A%3D%3D"
+			(at 105.41 644.45 0)
+			(effects
+				(font
+					(size 1.27 1.27)
+				)
+				(justify left top)
+				(hide yes)
+			)
+		)
+		(property "Manufacturer_Name" "Texas Instruments"
+			(at 105.41 744.45 0)
+			(effects
+				(font
+					(size 1.27 1.27)
+				)
+				(justify left top)
+				(hide yes)
+			)
+		)
+		(property "Manufacturer_Part_Number" "TLV6700DDCR"
+			(at 105.41 844.45 0)
+			(effects
+				(font
+					(size 1.27 1.27)
+				)
+				(justify left top)
+				(hide yes)
+			)
+		)
+		(pin "3"
+		)
+		(pin "4"
+		)
+		(pin "5"
+		)
+		(pin "6"
+		)
+		(pin "2"
+		)
+		(pin "1"
+		)
+		(instances
+			(project "c5_adapter"
+				(path "/4ea9e048-096c-4569-98b9-ff311a85c85d"
+					(reference "IC1")
+					(unit 1)
+				)
